File: TinyCoinCell.kicad_sch (KiCad schematic)
At the start: 47 parts, among them SW1 SW_Push, U1 nRF54L15-QFAA, U8 nPM2100-QEXX, X1 32MHz, X2 32.768kHz

Commit message: Update for nPM2100, ADXL367
Parts:
- added C48, C50, C51: 1uF, Capacitor_SMD:C_0201_0603Metric, symbol Device:C_Small
- added U2: ADXL367, TinyCoinCell:ADXL367_LGA-12_2.11x2.21mm_P0.5mm_LayoutBorder2x4y, symbol TinyCoinCell:ADXL367
- TP1, TP2, TP3, TP4, TP5, TP6, TP7: now in the parts list
Connections:
- net SCL: now also U2.4 (~{CS})
- net SDA: now also U2.2 (MOSI)
- net VDD: now also C48.1, C50.1, U2.10 (V_{S}), U2.12 (V_{DDIO})
- net INT1: now reaches U1.40 (P1.12)
- net INT1: now also U2.5 (INT1)
- net AVSS2 renamed GND
- net GND: now also U8.[11,16,17] (VSS), C48.2, C50.2, C51.2, U2.1 (SCLK), U2.11 (GND), U2.3 (MISO), U2.7 (GND); no longer U8.11 (AVSS2), U8.16 (PVSS), U8.17 (EP)
- new net: C51.1, U2.9 (V_{REG_OUT})
- no-connect marks 27 -> 28
Other:
- moved on the sheet: U8
